File: kicad/stlink.kicad_pcb (KiCad board)
At the start: 2 copper layers, 47.3 x 23.4 mm, 49 parts, among them J1 USB_A, J2 jtag, J3 boot0, J4 st_swdio, J5 st_swclk, J8 SWIM, J9 st_prog, U1 NCP603, U2 STM32F103C8Tx, Y1 8mgh

Commit message: start
Parts:
- added C14: 10n, Capacitors_SMD:C_0603_HandSoldering, B.Cu at (156.2, 72.3)
- U1: value NCP603 -> LDS3985M33R (NCP603)
- moved C5 2.69 mm to (155.2, 75.7), turned to 270 degrees
- moved C6 2.63 mm to (157.5, 75.6), turned to 270 degrees
Connections:
- U2 pad 1: VDD -> (no net)
- U2 pad 11: Net-(U2-Pad11) -> (no net)
- U2 pad 12: Net-(U2-Pad12) -> (no net)
- U2 pad 13: Net-(U2-Pad13) -> (no net)
- U2 pad 14: Net-(U2-Pad14) -> (no net)
- U2 pad 2: Net-(U2-Pad2) -> (no net)
- U2 pad 28: Net-(U2-Pad28) -> (no net)
- U2 pad 29: Net-(U2-Pad29) -> (no net)
- U2 pad 3: Net-(U2-Pad3) -> (no net)
- U2 pad 38: Net-(U2-Pad38) -> (no net)
- U2 pad 39: Net-(U2-Pad39) -> (no net)
- U2 pad 4: Net-(U2-Pad4) -> (no net)
- U2 pad 40: Net-(U2-Pad40) -> (no net)
Routing:
- net VDD: track 117.9 -> 114.9 mm
- net Net-(C14-Pad1): track 0.00 -> 2.50 mm
