File: kicad/stlink.sch (KiCad schematic (older format))
At the start: 49 parts, among them J1 USB_A, J2 jtag, J3 boot0, J4 st_swdio, J5 st_swclk, J8 SWIM, J9 st_prog, U1 NCP603, U2 STM32F103C8Tx, Y1 8mgh

Commit message: start
Parts:
- added C14: 10n, Capacitors_SMD:C_0603_HandSoldering, symbol stlink-rescue:C_Small
- C1, C10, C11, C12, C13, C2, C3, C4, C5, C6, C7, C8, C9: symbol C_Small -> stlink-rescue:C_Small
- D1, D2: symbol LED -> stlink-rescue:LED
- J1: symbol USB_A -> stlink-rescue:USB_A
- J2: symbol CONN_02X05 -> stlink-rescue:CONN_02X05
- J3, J4, J5: symbol CONN_01X01 -> stlink-rescue:CONN_01X01
- J8: symbol CONN_01X05 -> stlink-rescue:CONN_01X05
- J9: symbol CONN_01X02 -> stlink-rescue:CONN_01X02
- R1, R10, R11, R12, R13, R14, R15, R16, R17, R18, R19, R2, R20, R21, R22, R23, R24, R25, R26, R4, R5, R6, R8, R9: symbol R_Small -> stlink-rescue:R_Small
- U1: value NCP603 -> LDS3985M33R (NCP603); symbol NCP603 -> mylibkicad:NCP603
- U2: symbol STM32F103C8Tx -> stlink-rescue:STM32F103C8Tx
- Y1: symbol Crystal_Small -> stlink-rescue:Crystal_Small
Connections:
- net GND: now also C14.2
- net at U1.4 (NCP): now also C14.1
